Commit message: Updated description and blocked-out joint republisher

File: go1_biped_description/urdf/go1_biped.urdf.xacro (robot description, xacro)
@@ -1,7 +1,7 @@
 <?xml version="1.0"?>
 <robot xmlns:xacro="http://ros.org/wiki/xacro" name="go1_biped">
-  <link name="base_link" />
+  <xacro:include filename="$(find go1_description)/urdf/go1.urdf"/>
   <joint name="GV7_joint" type="fixed">
-    <parent link="base_link" />
+    <parent link="base" />
     <child link="sensor" />
     <origin xyz="0.2 0 0.1" rpy="0 0 0"/>

Commit message: Updated ekf so it's better

File: go1_biped_description/urdf/go1_biped.urdf.xacro (robot description, xacro)
@@ -5,5 +5,5 @@
     <parent link="base" />
     <child link="sensor" />
-    <origin xyz="0.2 0 0.1" rpy="0 0 0"/>
+    <origin xyz="0.2 0 0.1" rpy="3.14159 0 0"/>
   </joint>
   <link name="sensor" />
